Commit message: mesh finding

File: src/my_rover/urdf/ref.urdf (robot description, URDF)
Before this commit: robot rover, 18 links, 17 joints
Links:
- link Base_link: geometry collision mesh filename=file://$(find my_rover)/meshes/stl/Assem1.stl scale=0.00100 0.00100 0.00100; visual mesh filename=file://$(find my_rover)/meshes/stl/Assem1.stl scale=0.00100 0.00100 0.00100

Commit message: Added camera

File: src/my_rover/urdf/ref.urdf (robot description, URDF)
Before this commit: robot rover, 18 links, 17 joints
Links:
- added link camera_link
Joints:
- added joint camera_link_joint: type fixed, parent Base_link, child camera_link, origin xyz=0.10 0.0 0.05 rpy=-1.57060 -1.57057 0

Commit message: Added imu and lidar

File: src/my_rover/urdf/ref.urdf (robot description, URDF)
Before this commit: robot rover, 19 links, 18 joints
Links:
- added link lidar_link
Joints:
- added joint lidar_joint: type fixed, parent Base_link, child lidar_link, origin xyz=0.0 0.0 0.15 rpy=0 0 0

Commit message: Clock issue not solved

File: src/my_rover/urdf/ref.urdf (robot description, URDF)
Before this commit: robot rover, 20 links, 19 joints
Links:
- removed link Base_link
- added link base_link, mass 5.00000; collision mesh filename=file://$(find my_rover)/meshes/stl/Assem1.stl scale=0.00100 0.00100 0.00100; visual mesh filename=file://$(find my_rover)/meshes/stl/Assem1.stl scale=0.00100 0.00100 0.00100
Joints:
- joint BackLeftMotor_link_joint: parent Base_link -> base_link
- joint BackRightMotor_link_joint: parent Base_link -> base_link
- joint FrontLeftMotor_link_joint: parent Base_link -> base_link
- joint FrontRightMotor_link_joint: parent Base_link -> base_link
- joint Stand1_link_joint: parent Base_link -> base_link
- joint Stand2_link_joint: parent Base_link -> base_link
- joint Stand3_link_joint: parent Base_link -> base_link
- joint Stand4_link_joint: parent Base_link -> base_link
- joint Stand5_link_joint: parent Base_link -> base_link
- joint Stand6_link_joint: parent Base_link -> base_link
- joint Stand7_link_joint: parent Base_link -> base_link
- joint Stand9_link_joint: parent Base_link -> base_link
- joint UpperBaseplate_link_joint: parent Base_link -> base_link
- joint camera_link_joint: parent Base_link -> base_link
- joint lidar_joint: parent Base_link -> base_link
